File: Transflective/LCD-Panel/LCD-panel.sch (KiCad schematic (older format))
At the start: 35 parts, among them J1 Conn_02x06_Odd_Even, J2 DS BACKLIGHT, U1 CAP1298

Commit message: Reorganize Transflective directories
Parts:
- gave numbers to parts that had none: 6
Changed lines of the file:
@@
 NoConn ~ 2950 3800
 $Comp
-L Transflective:ADP1650 U?
+L Transflective:ADP1650 U2
 U 1 1 616E8478
 P 3600 5900
-F 0 "U?" H 3875 6175 50  0000 C CNN
+F 0 "U2" H 3875 6175 50  0000 C CNN
 F 1 "ADP1650" H 3875 6084 50  0000 C CNN
 F 2 "" H 3600 5900 50  0001 C CNN
@@
 $EndComp
 $Comp
-L Device:CP1_Small C?
+L Device:CP1_Small C15
 U 1 1 616E857E
 P 5050 6100
-F 0 "C?" V 5278 6100 50  0000 C CNN
+F 0 "C15" V 5278 6100 50  0000 C CNN
 F 1 "10uF" V 5187 6100 50  0000 C CNN
 F 2 "Capacitor_SMD:C_0805_2012Metric_Pad1.15x1.40mm_HandSolder" H 5050 6100 50  0001 C CNN
@@
 $EndComp
 $Comp
-L Device:CP1_Small C?
+L Device:CP1_Small C14
 U 1 1 616E8730
 P 5050 5850
-F 0 "C?" V 5278 5850 50  0000 C CNN
+F 0 "C14" V 5278 5850 50  0000 C CNN
 F 1 "C10uF" V 5187 5850 50  0000 C CNN
 F 2 "Capacitor_SMD:C_0805_2012Metric_Pad1.15x1.40mm_HandSolder" H 5050 5850 50  0001 C CNN
@@
 $EndComp
 $Comp
-L power:GND #PWR?
+L power:GND #PWR0108
 U 1 1 616E8792
 P 4650 6550
-F 0 "#PWR?" H 4650 6300 50  0001 C CNN
+F 0 "#PWR0108" H 4650 6300 50  0001 C CNN
 F 1 "GND" H 4655 6377 50  0000 C CNN
 F 2 "" H 4650 6550 50  0001 C CNN
@@
 $EndComp
 $Comp
-L power:GND #PWR?
+L power:GND #PWR0109
 U 1 1 616E87DD
 P 5200 6100
-F 0 "#PWR?" H 5200 5850 50  0001 C CNN
+F 0 "#PWR0109" H 5200 5850 50  0001 C CNN
 F 1 "GND" H 5205 5927 50  0000 C CNN
 F 2 "" H 5200 6100 50  0001 C CNN
@@
 $EndComp
 $Comp
-L power:GND #PWR?
+L power:GND #PWR0110
 U 1 1 616E8828
 P 7750 6500
-F 0 "#PWR?" H 7750 6250 50  0001 C CNN
+F 0 "#PWR0110" H 7750 6250 50  0001 C CNN
 F 1 "GND" H 7755 6327 50  0000 C CNN
 F 2 "" H 7750 6500 50  0001 C CNN
@@
 	7750 6300 7750 5850
 $Comp
-L Device:L_Small L?
+L Device:L_Small L1
 U 1 1 616F3E5F
 P 4750 5950
-F 0 "L?" V 4935 5950 50  0000 C CNN
+F 0 "L1" V 4935 5950 50  0000 C CNN
 F 1 "1.0uH" V 4844 5950 50  0000 C CNN
 F 2 "" H 4750 5950 50  0001 C CNN
@@
 	4850 5850 4950 5850
 $Comp
-L power:+3.3V #PWR?
+L power:+3.3V #PWR0111
 U 1 1 61718FAB
 P 4850 5650
-F 0 "#PWR?" H 4850 5500 50  0001 C CNN
+F 0 "#PWR0111" H 4850 5500 50  0001 C CNN
 F 1 "+3.3V" H 4865 5823 50  0000 C CNN
 F 2 "" H 4850 5650 50  0001 C CNN
@@
 	3200 6250 2850 6250
 $Comp
-L power:GND #PWR?
+L power:GND #PWR0112
 U 1 1 6173B6C1
 P 2700 6100
-F 0 "#PWR?" H 2700 5850 50  0001 C CNN
+F 0 "#PWR0112" H 2700 5850 50  0001 C CNN
 F 1 "GND" H 2705 5927 50  0000 C CNN
 F 2 "" H 2700 6100 50  0001 C CNN
@@
 	3200 6100 2700 6100
 $Comp
-L Connector:TestPoint TP?
+L Connector:TestPoint TP7
 U 1 1 61751766
 P 3150 5850
-F 0 "TP?" V 3345 5924 50  0000 C CNN
+F 0 "TP7" V 3345 5924 50  0000 C CNN
 F 1 "TestPoint" V 3254 5924 50  0000 C CNN
 F 2 "TestPoint:TestPoint_Pad_D1.0mm" H 3350 5850 50  0001 C CNN
@@
 $EndComp
 $Comp
-L Connector:TestPoint TP?
+L Connector:TestPoint TP8
 U 1 1 6175180E
 P 3150 5950
-F 0 "TP?" V 3345 6024 50  0000 C CNN
+F 0 "TP8" V 3345 6024 50  0000 C CNN
 F 1 "TestPoint" V 3254 6024 50  0000 C CNN
 F 2 "TestPoint:TestPoint_Pad_D1.0mm" H 3350 5950 50  0001 C CNN

Commit message: Front panel functionally complete
Still to do: verify orientation of LCD pinout, add 3.3V regulator option
Parts:
- removed U2: ADP1650, symbol Transflective:ADP1650
- added JP5: LED PWR, Jumper:SolderJumper-3_P1.3mm_Bridged12_RoundedPad1.0x1.5mm, symbol Jumper:SolderJumper_3_Bridged12
- added TP9: TestPoint, TestPoint:TestPoint_Pad_D1.0mm, symbol Connector:TestPoint
- added U2: ADP1650ACPZ-R7, ADP1650:ADP1650ACPZ-R7, symbol ADP1650:ADP1650ACPZ-R7
- C14: value C10uF -> 10uF
- J1: footprint Connector_IDC:IDC-Header_2x06_P2.54mm_Vertical -> Connector_PinHeader_2.54mm:PinHeader_2x07_P2.54mm_Vertical_SMD; symbol Connector_Generic:Conn_02x06_Odd_Even -> Connector_Generic:Conn_02x07_Odd_Even
- L1: footprint (none) -> Inductor_SMD:L_0805_2012Metric_Pad1.15x1.40mm_HandSolder
Connections:
- net labels added: +5V
- wire segments 150 -> 163
Other:
- note added: "Add 3.3V regulator"
- note removed: "Add ADP1650ACPZ-R7 to drive backlight LED"

Commit message: The FPC connector was mirrored :(
Add a vertical FPC connector, with the proper orienatation.  A bunch of
stuff needs to be rerouted.
Parts:
- DS1: footprint Connector_FFC-FPC:Hirose_FH12-36S-0.5SH_1x36-1MP_P0.50mm_Horizontal -> Transflective:F314-1A7H1-11036
Changed lines of the file:
@@
 F 0 "DS1" H 9128 -404 50  0000 L CNN
 F 1 "DISPLAYTECH-128240D" H 9128 -495 50  0000 L CNN
-F 2 "Connector_FFC-FPC:Hirose_FH12-36S-0.5SH_1x36-1MP_P0.50mm_Horizontal" H 8200 1550 50  0001 C CNN
+F 2 "Transflective:F314-1A7H1-11036" H 8200 1550 50  0001 C CNN
 F 3 "" H 8200 1550 50  0001 C CNN
 	1    8200 1550

Commit message: Reroute the FPC connector
Changed lines of the file:
@@
 	1400 1550 2200 1550
 Wire Wire Line
-	1400 1650 2200 1650
+	1400 1350 2200 1350
 Wire Wire Line
 	2700 1550 3500 1550
@@
 	1400 1450 2200 1450
 Wire Wire Line
-	1400 1350 2200 1350
+	1400 1650 2200 1650
 Text Label 3150 1450 0    50   ~ 0
 CAP_CLK
@@
 Text Label 1400 1550 0    50   ~ 0
 DS_DAT
+Text Label 1400 1650 0    50   ~ 0
+DS_CS
 Text Label 1400 1350 0    50   ~ 0
-DS_CS
-Text Label 1400 1650 0    50   ~ 0
 DS_RST
 $Comp

Commit message: Finish designing front and rear boards for Transflective LCD version
Parts:
- added C16: .1uF, Capacitor_SMD:C_0805_2012Metric_Pad1.15x1.40mm_HandSolder, symbol Device:CP1_Small
- added C17: .01uF, Capacitor_SMD:C_0805_2012Metric_Pad1.15x1.40mm_HandSolder, symbol Device:CP1_Small
- added C18: 1uF, Capacitor_SMD:C_0805_2012Metric_Pad1.15x1.40mm_HandSolder, symbol Device:CP1_Small
- added J3, J4: STEMMA I2C QT, Transflective:JST-SH-4-VERT-SMD, symbol Connector_Generic:Conn_01x04
- added JP6: USE LOCAL REG, Jumper:SolderJumper-3_P1.3mm_Bridged12_RoundedPad1.0x1.5mm, symbol Jumper:SolderJumper_3_Bridged12
- added R3, R4: 10k, Resistor_SMD:R_0805_2012Metric_Pad1.15x1.40mm_HandSolder, symbol Device:R_Small_US
- added U3: AP131-33, Package_TO_SOT_SMD:SOT-23-5, symbol Regulator_Linear:AP131-33
- J1: value Conn_02x06_Odd_Even -> To Bottom Board
- TP1: value TestPoint -> GUARD
- TP2: value TestPoint -> A
- TP3: value TestPoint -> B
- TP4: value TestPoint -> C
- TP5: value TestPoint -> D
- TP6: value TestPoint -> PROX
- TP7: value TestPoint -> GPIO1
- TP8: value TestPoint -> GPIO2
- TP9: value TestPoint -> Unused
Connections:
- wire segments 163 -> 198
