File: Transflective/Rear-Panel/Transflective.sch (KiCad schematic (older format))
At the start: 5 parts, among them J1 feather long, J2 feather short, J3 feather long, J4 feather short, U1 Pico

Commit message: Reorganize Transflective directories
Parts:
- added J5: PermaProto, Transflective:PermaProto, symbol Transflective:PermaProto
Changed lines of the file:
@@
 Text Notes 5050 5150 0    50   ~ 0
 ADC board (outside)
+$Comp
+L Transflective:PermaProto J5
+U 1 1 6152F3A3
+P 9250 4900
+F 0 "J5" H 9528 4846 50  0000 L CNN
+F 1 "PermaProto" H 9528 4755 50  0000 L CNN
+F 2 "Transflective:PermaProto" H 9250 4900 50  0001 C CNN
+F 3 "" H 9250 4900 50  0001 C CNN
+	1    9250 4900
+	1    0    0    -1
+$EndComp
 $EndSCHEMATC

Commit message: Finish designing front and rear boards for Transflective LCD version
Parts:
- added D1: D_Schottky, Diode_THT:D_DO-41_SOD81_P10.16mm_Horizontal, symbol Device:D_Schottky
- added J10: STEMMA QT, Connector_JST:JST_XH_B04B-XH-AM_1x04_P2.50mm_Vertical, symbol Connector_Generic:Conn_01x04
- added J11: LCD CS, Connector_JST:JST_XH_B03B-XH-AM_1x03_P2.50mm_Vertical, symbol Connector:Conn_01x03_Female
- added J12: WATER, Connector_JST:JST_XH_B03B-XH-AM_1x03_P2.50mm_Vertical, symbol Connector:Conn_01x03_Female
- added J13: PUMP, Connector_JST:JST_XH_B03B-XH-AM_1x03_P2.50mm_Vertical, symbol Connector:Conn_01x03_Female
- added J14: MISO, Connector_PinHeader_2.54mm:PinHeader_1x01_P2.54mm_Vertical, symbol Connector:Conn_01x01_Female
- added J15: CAP ALERT, Connector_PinHeader_2.54mm:PinHeader_1x01_P2.54mm_Vertical, symbol Connector:Conn_01x01_Female
- added J16: PRESSURE, Connector_JST:JST_XH_B03B-XH-AM_1x03_P2.50mm_Vertical, symbol Connector:Conn_01x03_Female
- added J17: Pressure Switch, Connector_JST:JST_XH_B02B-XH-AM_1x02_P2.50mm_Vertical, symbol Connector:Conn_01x02_Female
- added J18: PowerTail Out, Connector_JST:JST_XH_B02B-XH-AM_1x02_P2.50mm_Vertical, symbol Connector:Conn_01x02_Female
- added J19: UNUSED, Connector_PinHeader_2.54mm:PinHeader_1x01_P2.54mm_Vertical, symbol Connector:Conn_01x01_Female
- added J6: To LCD Board, Connector_IDC:IDC-Header_2x07_P2.54mm_Vertical, symbol Connector_Generic:Conn_02x07_Odd_Even
- added J7: SNITCH, Connector_JST:JST_XH_B03B-XH-AM_1x03_P2.50mm_Vertical, symbol Connector:Conn_01x03_Female
- added J8, J9: STEMMA QT, Transflective:JST-SH-4-VERT-SMD, symbol Connector_Generic:Conn_01x04
- added JP1: LCD CS, Jumper:SolderJumper-3_P1.3mm_Bridged2Bar12_RoundedPad1.0x1.5mm, symbol Jumper:SolderJumper_3_Bridged12
- added R1, R2, R3: 10k, Resistor_THT:R_Axial_DIN0207_L6.3mm_D2.5mm_P10.16mm_Horizontal, symbol Device:R_Small_US
- added U2: 74LVC1G02, Package_TO_SOT_SMD:SOT-23-5_HandSoldering, symbol 74xGxx:74LVC1G02
Connections:
- net labels added: +5V, CAP_ALERT, DS_CS, SNITCH_3V3, SNITCH_SIG, VCC
- wire segments 60 -> 159
- no-connect marks 0 -> 8
Other:
- note added: "ADC"
- note added: "LED0"
- note added: "LED1"
- note added: "MISO"
- note added: "MOSI"
- note added: "NC"
- note added: "SCK"
- note removed: "5V / 12V input/output"
- note removed: "ADC board (outside)"
- note removed: "ST7529 FPC"

Commit message: Some notes about errata discovered in the v1 PCBs, and BOMs
Other:
- note added: "XXX: This should be a 3.3V supply to U2"
Changed lines of the file:
@@
 	1    0    0    -1
 $EndComp
+Text Notes 2900 4200 0    50   ~ 0
+XXX: This should be a 3.3V supply to U2
 $EndSCHEMATC
