File: Transflective/Snitch-2/Snitch-2.kicad_pcb (KiCad board)
At the start: 2 copper layers, 80.5 x 29.2 mm, 35 parts, among them J1 SNITCH IN, J2 To Pico, U1 AMC23C10, U2 AMC23C10

Commit message: Snitch PCB and BOM
Other:
- board text added: "JLCJLCJLCJLC"
